File: pcb/dendrite/dendrite.kicad_pcb (KiCad board)
At the start: 2 copper layers, 264.5 x 31.3 mm, 29 parts, among them J1 Conn_01x25, J10 Conn_01x13, J11 Conn_01x13, J12 Conn_01x13, J13 Conn_01x13, J14 Conn_01x13, J15 Conn_01x13, J16 Conn_01x13, J17 Conn_01x13, J2 Conn_01x13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

Commit message: extending the cable
Parts:
- moved G*** 39.3 mm to (124.0, 41.9)
- moved G*** 39.3 mm to (124.0, 42.1)
- moved J1 39.3 mm to (115.0, 42.0)
- moved JP7 37.7 mm to (76.0, 25.9)
- moved JP10 37.7 mm to (37.0, 15.8)
- moved JP6 37.7 mm to (36.8, 25.9)
- moved JP5 37.7 mm to (1.91, 25.9)
- moved JP9 37.7 mm to (1.91, 16.0)
- moved JP8 37.7 mm to (108.3, 20.3)
- moved J7 21.9 mm to (43.2, 9.59)
- moved J4 21.7 mm to (156.4, 9.59)
- moved J6 21.6 mm to (80.6, 9.60)
- moved J5 21.5 mm to (118.4, 9.60)
- moved J17 18.1 mm to (-7.87, 30.8)
- moved J13 18.1 mm to (-7.86, 21.0)
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Routing:
- net GND: track 962.4 -> 1345.2 mm
- net +5V: track 946.5 -> 1327.4 mm
- net row0: track 610.5 -> 869.2 mm
- net row1: track 509.9 -> 684.0 mm
- net row3: track 519.8 -> 693.7 mm
- net row2: track 478.4 -> 652.1 mm
- net row5: track 441.9 -> 615.5 mm
- net row6: track 437.4 -> 610.8 mm
- net row4: track 426.9 -> 578.4 mm
- net col2: track 365.7 -> 501.1 mm
- net col3: track 364.1 -> 495.8 mm
- net col5: track 536.4 -> 667.3 mm
- net col4: track 518.7 -> 648.7 mm
- net col6: track 525.4 -> 647.5 mm
- net col7: track 481.6 -> 601.6 mm
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Other:
- board size 264.5 x 31.3 mm -> 265.1 x 45.8 mm
